Commit message: Add files via upload
SImulation with lidar working but have a little issue with the angles

File: charmie_bot/description/robot.urdf.xacro (robot description, xacro)
@@ -1,5 +1,7 @@
 <?xml version="1.0"?>
 <robot xmlns:xacro="http://www.ros.org/wiki/xacro"  name="robot">
-    <!--Example Link-->
-    <link name='base_link'/>
+    <xacro:include filename='robot_core.xacro'/>
+    <xacro:include filename='robot_wheels.xacro'/>
+    <xacro:include filename='gazebo_control.xacro'/>
+    <xacro:include filename='lidar.xacro'/>
 </robot>
