Commit message: Simulation with LIDAR and JOYSTICK OK

File: charmie_bot/description/lidar.xacro (robot description, xacro)
@@ -1,17 +1,17 @@
 <?xml version="1.0"?>
-<robot xmlns:xacro="http://www.ros.org/wiki/xacro">
-    <joint name="lidar_joint" type="fixed">
-        <parent link="base_link"/>
-        <child link="lidar_frame"/>
-        <origin xyz="0.2 0 0.21" rpy="0 0 0"/>
+<robot xmlns:xacro="http://www.ros.org/wiki/xacro" >
+    <joint name="laser_joint" type="fixed">
+        <parent link="chassi_link"/>
+        <child link="laser_frame"/>
+        <origin xyz="0.2 0 0.177" rpy="0 0 0"/>
     </joint>
-    <link name="lidar_frame">
+    <link name="laser_frame">
         <visual>
-            <origin xyz="0 0 0" rpy="0 0 0"/>
+            <origin xyz="0 0 -0.055" rpy="${pi/2} 0 ${pi}"/>
             <geometry>
-                <!-- <mesh filename="file://$(find charmie_bot)/description/meshes/lidar.stl" scale="0.001 0.001 0.001"/> -->
-                <cylinder radius="0.05" length="0.04"/>
+                <mesh filename="file://$(find charmie_bot)/description/meshes/lidar.stl" scale="0.001 0.001 0.001"/>
+                <!-- <cylinder radius="0.05" length="0.04"/> -->
             </geometry>
-            <material name="black"/>
+            <material name="red"/>
         </visual>
         <collision>
@@ -24,8 +24,8 @@
         </xacro:inertial_cylinder>
     </link>
-    <gazebo reference="lidar_frame">
-        <material>Gazebo/Black</material>
+    <gazebo reference="laser_frame">
+        <material>Gazebo/Red</material>
         <sensor name="laser" type="ray">
-            <pose>0 0 0 0 0 0</pose>
+            <pose> 0 0 0.055 0 0 0 </pose>
             <visualize>true</visualize>
             <update_rate>10</update_rate>
@@ -33,6 +33,6 @@
                 <scan>
                     <horizontal>
-                        <samples>360</samples> <!--681-->
-                        <min_angle>-2.092387973753402</min_angle> <!--19.8 degrees 2.092387973753402 rad-->
+                        <samples>681</samples>
+                        <min_angle>-2.092387973753402</min_angle>
                         <max_angle>2.092387973753402</max_angle>
                     </horizontal>
@@ -48,5 +48,5 @@
                 </ros>
                 <output_type>sensor_msgs/LaserScan</output_type>
-                <frame_name>lidar_frame</frame_name>
+                <frame_name>laser_frame</frame_name>
             </plugin>
         </sensor>

File: charmie_bot/description/robot.urdf.xacro (robot description, xacro)
@@ -1,7 +1,7 @@
 <?xml version="1.0"?>
-<robot xmlns:xacro="http://www.ros.org/wiki/xacro"  name="robot">
+<robot xmlns:xacro="http://www.ros.org/wiki/xacro"  name="charmie_robot">
     <xacro:include filename='robot_core.xacro'/>
     <xacro:include filename='robot_wheels.xacro'/>
+    <xacro:include filename='lidar.xacro'/>
     <xacro:include filename='gazebo_control.xacro'/>
-    <xacro:include filename='lidar.xacro'/>
 </robot>

File: charmie_bot/description/robot_core.xacro (robot description, xacro)
@@ -35,5 +35,5 @@
         </visual>
         <collision>
-            <origin xyz="0 0 0.085"/>
+            <origin xyz="0 0 0"/>
             <geometry>
                 <cylinder radius="0.275" length="0.25"/>
@@ -41,5 +41,5 @@
         </collision>
         <xacro:inertial_cylinder mass="1.0" length="0.25" radius="0.275">
-            <origin xyz="0 0 0.085" rpy="0 0 0"/>
+            <origin xyz="0 0 0" rpy="0 0 0"/>
         </xacro:inertial_cylinder>
     </link>
