Commit message: Adding the SLAM_TOOLBOX and NAV2

File: charmie_bot/description/robot_core.xacro (robot description, xacro)
@@ -19,4 +19,12 @@
     <!--BASE LINK-->
     <link name="base_link">
+    </link>
+    <!--BASE FOOTPRINT-->
+    <joint name="base_footprint_joint" type="fixed">
+        <parent link="base_link"/>
+        <child link="base_footprint"/>
+        <origin xyz="0 0 0" rpy="0 0 0"/>
+    </joint>
+    <link name="base_footprint">
     </link>
     <!--CHASSI-->
